Commit message: construct motor position

File: urdf/simbicon_urdf/flame.urdf (robot description, URDF)
Before this commit: robot humanoid, 12 links, 10 joints
Links:
- added link lowerLegBridgeR, mass 0.267; collision box size=0.1 0.05 0.28; visual box size=0.1 0.05 0.28
- added link upperLegBridgeR, mass 1.94; collision box size=0.1 0.05 0.3155; visual box size=0.1 0.05 0.3155
Joints:
- added joint fixed_hipBridgeR: type fixed, parent hipCylinderR, child hipBridgeR
- added joint fixed_lowerLegBridgeR: type fixed, parent lowerlegCylinderR, child lowerLegBridgeR
- added joint fixed_upperLegBridgeR: type fixed, parent upperLegCylinderR, child upperLegBridgeR
- joint jointHipL: axis 0 0 1 -> 1 0 0
- joint jointHipR: axis 0 0 1 -> 1 0 0
- joint jointUpperLegL: axis 1 0 0 -> 0 1 0
- joint jointUpperLegR: axis 1 0 0 -> 0 1 0
- joint jointfootL: axis 0 1 0 -> 1 0 0
- joint jointfootR: axis 0 1 0 -> 1 0 0

Commit message: construct shape

File: urdf/simbicon_urdf/flame.urdf (robot description, URDF)
Before this commit: robot humanoid, 14 links, 13 joints
Links:
- added link ankleBridgeL, mass 0.2356; collision box size=0.1 0.05 0.02; visual box size=0.1 0.05 0.02
- added link ankleBridgeR, mass 0.2356; collision box size=0.1 0.05 0.02; visual box size=0.1 0.05 0.02
- added link hipBridgeL, mass 0.219; collision box size=0.02 0.0830 0.0250; visual box size=0.02 0.0830 0.0250
- added link lowerLegBridgeL, mass 0.267; collision box size=0.1 0.05 0.28; visual box size=0.1 0.05 0.28
- added link upperLegBridgeL, mass 1.94; collision box size=0.1 0.05 0.3155; visual box size=0.1 0.05 0.3155
Joints:
- added joint fixed_ankleBridgeL: type fixed, parent ankleCylinderL, child ankleBridgeL
- added joint fixed_ankleBridgeR: type fixed, parent ankleCylinderR, child ankleBridgeR
- added joint fixed_hipBridgeL: type fixed, parent hipCylinderL, child hipBridgeL
- added joint fixed_lowerLegBridgeL: type fixed, parent lowerlegCylinderL, child lowerLegBridgeL
- added joint fixed_upperLegBridgeL: type fixed, parent upperLegCylinderL, child upperLegBridgeL

Commit message: add body part

File: urdf/simbicon_urdf/flame.urdf (robot description, URDF)
Before this commit: robot humanoid, 19 links, 18 joints
Links:
- removed link footCylinderL
- removed link footCylinderR
- added link body, mass 5.6; collision box size=0.05 0.2 0.3; visual box size=0.05 0.2 0.3
- link ankleBridgeL: geometry collision box size=0.16 0.13 0.02; visual box size=0.16 0.13 0.02
- link ankleBridgeR: geometry collision box size=0.16 0.13 0.02; visual box size=0.16 0.13 0.02
- link lowerLegBridgeL: geometry collision box size=0.05 0.05 0.28; visual box size=0.05 0.05 0.28
- link lowerLegBridgeR: geometry collision box size=0.05 0.05 0.28; visual box size=0.05 0.05 0.28
- link torso: mass 0 -> 1.0
Joints:
- removed joint jointfootL
- removed joint jointfootR
- added joint torsoBody: type fixed, parent torso, child body
- joint jointAnkleL: origin xyz=0.00300 0 -0.28 rpy=0 0 0 -> xyz=0.00300 0 -0.2915 rpy=0 0 0
- joint jointAnkleR: origin xyz=0.00300 0 -0.28 rpy=0 0 0 -> xyz=0.00300 0 -0.2915 rpy=0 0 0
