Commit message: fix inertia and initial condition

File: urdf/simbicon_urdf/flame2.urdf (robot description, URDF)
Before this commit: robot humanoid, 18 links, 17 joints
Links:
- link body: mass 5.6 -> 10.14
- link torso: mass 1.0 -> 0.0
Joints:
- joint jointAnkleR: origin xyz=0.00300 0 -0.2915 rpy=0 0 0 -> xyz=0.00300 0 -0.2915 rpy=-0.021 0.164 0
- joint jointHipL: origin xyz=0 0.0 0.0 rpy=0 0 0 -> xyz=0 0.0 0.0 rpy=0 -0.1 0
- joint jointHipR: origin xyz=0 0.0 0.0 rpy=0 0 0 -> xyz=0 0.0 0.0 rpy=0 -0.1 0
