Commit message: add trajs and flame3

File: urdf/simbicon_urdf/flame3.urdf (robot description, URDF)
Before this commit: robot humanoid, 18 links, 17 joints
Links:
- link body: mass 10.14 -> 5.6
- link torso: mass 0.0 -> 1.0
Joints:
- joint jointAnkleR: origin xyz=0.00300 0 -0.2915 rpy=-0.021 0.164 0 -> xyz=0.00300 0 -0.2915 rpy=0 0 0
- joint jointHipL: origin xyz=0 0.0 0.0 rpy=0 -0.1 0 -> xyz=0 0.0 0.0 rpy=0 0 0
- joint jointHipR: origin xyz=0 0.0 0.0 rpy=0 -0.1 0 -> xyz=0 0.0 0.0 rpy=0 0 0
- joint jointUpperLegL: origin xyz=0 0.0830 -0.0250 rpy=0 -0.994 0 -> xyz=0 0.0830 -0.0250 rpy=0 -0.5 0
- joint torsoBody: origin xyz=0 0.0 0.0 rpy=-0.0056 -0.0021 0 -> xyz=0 0.0 -0.15 rpy=0.0 0.0 0; type revolute -> fixed

Commit message: controller

File: urdf/simbicon_urdf/flame3.urdf (robot description, URDF)
Before this commit: robot humanoid, 18 links, 17 joints
Joints:
- joint torsoBody: axis 0 1 0 -> 1 0 0; child torso -> body; origin xyz=0 0.0 -0.15 rpy=0.0 0.0 0 -> xyz=0 0.0 0 rpy=0.0 0.0 0; parent body -> torso

Commit message: Update flame3.urdf

File: urdf/simbicon_urdf/flame3.urdf (robot description, URDF)
Before this commit: robot humanoid, 18 links, 17 joints
Joints:
- joint jointAnkleL: limit lower=-3 upper=+3 effort=10 velocity=10 -> lower=-0.436332 upper=+0.436332 effort=90 velocity=10
- joint jointAnkleR: limit lower=-3 upper=+3 effort=10 velocity=10 -> lower=-0.436332 upper=+0.436332 effort=90 velocity=10
- joint jointHipL: limit lower=-3 upper=+3 effort=10 velocity=10 -> lower=0 upper=+0.174533 effort=90 velocity=10
- joint jointHipR: limit lower=-3 upper=+3 effort=10 velocity=10 -> lower=-0.174533 upper=0 effort=90 velocity=10
- joint jointLowerLegL: limit lower=-3 upper=+3 effort=10 velocity=10 -> lower=-1.570796 upper=0 effort=90 velocity=10
- joint jointLowerLegR: limit lower=-3 upper=+3 effort=10 velocity=10 -> lower=-1.570796 upper=0 effort=90 velocity=10
- joint jointUpperLegL: limit lower=-3 upper=+3 effort=10 velocity=10 -> lower=-0.174533 upper=+0.174533 effort=10 velocity=10
- joint jointUpperLegR: limit lower=-3 upper=+3 effort=10 velocity=10 -> lower=-0.698132 upper=+1.047 effort=90 velocity=10

Commit message: knees bend in right way

File: urdf/simbicon_urdf/flame3.urdf (robot description, URDF)
Before this commit: robot humanoid, 18 links, 17 joints
Joints:
- joint jointLowerLegL: limit lower=-1.570796 upper=0 effort=90 velocity=10 -> lower=0 upper=1.570796 effort=90 velocity=10
- joint jointLowerLegR: limit lower=-1.570796 upper=0 effort=90 velocity=10 -> lower=0 upper=1.570796 effort=90 velocity=10

Commit message: add upper leg motor into urdf

File: urdf/simbicon_urdf/flame3.urdf (robot description, URDF)
Before this commit: robot humanoid, 18 links, 17 joints
Links:
- added link Left_Motor1_gear; visual mesh filename=meshes/gear.obj scale=0.03 0.03 0.03
- added link Left_Motor1_motor; visual mesh filename=meshes/motor.obj scale=0.03 0.03 0.03
- added link Left_Motor2_gear; visual mesh filename=meshes/gear.obj scale=0.03 0.03 0.03
- added link Left_Motor2_motor; visual mesh filename=meshes/motor.obj scale=0.03 0.03 0.03
- added link Right_Motor1_gear; visual mesh filename=meshes/gear.obj scale=0.03 0.03 0.03
- added link Right_Motor1_motor; visual mesh filename=meshes/motor.obj scale=0.03 0.03 0.03
- added link Right_Motor2_gear; visual mesh filename=meshes/gear.obj scale=0.03 0.03 0.03
- added link Right_Motor2_motor; visual mesh filename=meshes/motor.obj scale=0.03 0.03 0.03
Joints:
- added joint fixed_Motor1_GearToMotor1_Motor: type fixed, parent Left_Motor1_gear, child Left_Motor1_motor, origin xyz=0 0 -0.08 rpy=0 0 0
- added joint fixed_Motor2_GearToMotor2_Motor: type fixed, parent Left_Motor2_gear, child Left_Motor2_motor, origin xyz=0 0 -0.08 rpy=0 0 0
- added joint fixed_Right_Motor1_GearToRight_Motor1_Motor: type fixed, parent Right_Motor1_gear, child Right_Motor1_motor, origin xyz=0 0 -0.08 rpy=0 0 0
- added joint fixed_Right_Motor2_GearToRight_Motor2_Motor: type fixed, parent Right_Motor2_gear, child Right_Motor2_motor, origin xyz=0 0 -0.08 rpy=0 0 0
- added joint fixed_RightupperLegToRight_Motor2_Gear: type fixed, parent upperLegCylinderR, child Right_Motor2_gear, origin xyz=0 -0.02 -0.1 rpy=0 0 0
- added joint fixed_upperLegToMotor1_Gear: type fixed, parent upperLegCylinderL, child Left_Motor1_gear, origin xyz=0 0.02 -0.1 rpy=0 0 0
- added joint fixed_upperLegToMotor2_Gear: type fixed, parent upperLegCylinderL, child Left_Motor2_gear, origin xyz=0 -0.02 -0.1 rpy=0 0 0
- added joint fixed_upperRightLegToRight_Motor1_Gear: type fixed, parent upperLegCylinderR, child Right_Motor1_gear, origin xyz=0 0.02 -0.1 rpy=0 0 0

Commit message: add ankle motor mesh preparing for SEA control

File: urdf/simbicon_urdf/flame3.urdf (robot description, URDF)
Before this commit: robot humanoid, 26 links, 25 joints
Links:
- added link Left_AnkleMotor_Gear; visual mesh filename=meshes/gear.obj scale=0.03 0.03 0.03
- added link Left_Ankle_motor; visual mesh filename=meshes/motor.obj scale=0.03 0.03 0.03
- added link Right_AnkleMotor_Gear; visual mesh filename=meshes/gear.obj scale=0.03 0.03 0.03
- added link Right_Ankle_motor; visual mesh filename=meshes/motor.obj scale=0.03 0.03 0.03
Joints:
- added joint fixed_Left_AnkleMotor_GearToLeft_Ankle_motor: type fixed, parent Left_AnkleMotor_Gear, child Left_Ankle_motor, origin xyz=0 0 -0.08 rpy=0 0 0
- added joint fixed_Right_AnkleMotor_GearToRight_Ankle_motor: type fixed, parent Right_AnkleMotor_Gear, child Right_Ankle_motor, origin xyz=0 0 -0.08 rpy=0 0 0
- added joint fixed_lowerLegBridgeLToLeft_AnkleMotor_Gear: type fixed, parent lowerLegBridgeL, child Left_AnkleMotor_Gear, origin xyz=0 0.02 -0.05 rpy=0 0 0
- added joint fixed_lowerLegBridgeRToRight_AnkleMotor_Gear: type fixed, parent lowerLegBridgeR, child Right_AnkleMotor_Gear, origin xyz=0 0.02 -0.05 rpy=0 0 0
