Commit message: backup

File: urdf/simbicon_urdf/biped2d.urdf (robot description, URDF)
Before this commit: robot balance, 10 links, 9 joints
Links:
- removed link y_prismatic
- removed link z_prismatic
Joints:
- removed joint y_to_world
- removed joint z_to_y
- joint torso_to_z: parent z_prismatic -> world
