Commit message: add 2d robot env

File: urdf/simbicon_urdf/flame_2d.urdf (robot description, URDF)
Before this commit: robot humanoid, 21 links, 20 joints
Links:
- removed link torso
- removed link y_prismatic
- added link x_prismatic, mass 0.01
Joints:
- removed joint torsoBody
- removed joint y_to_world
- added joint x_to_world: type prismatic, parent world, child x_prismatic, origin xyz=0 0 0 rpy=0 0 0, axis 1 0 0, limit lower=10 upper=-10 effort=0.0 velocity=1000.0
- joint jointHipL: parent torso -> body
- joint jointHipR: parent torso -> body
- joint torso_to_z: axis 1 0 0 -> 0 1 0; limit (none) -> lower=10 upper=-10 effort=0.0 velocity=1000.0; origin xyz=0 0 1.4 rpy=0 0 0 -> xyz=0 0 0 rpy=0 0 0; type continuous -> revolute
- joint z_to_y: limit lower=1 upper=-1 effort=0.0 velocity=1000.0 -> lower=10 upper=-10 effort=0.0 velocity=1000.0; parent y_prismatic -> x_prismatic
