Commit message: trajectory

File: urdf/simbicon_urdf/flame5.urdf (robot description, URDF)
Before this commit: robot humanoid, 20 links, 19 joints
Joints:
- joint jointUpperLegL: limit lower=-0.174533 upper=+0.174533 effort=10 velocity=10 -> lower=-0.523599 upper=+1.22173 effort=10 velocity=10
- joint jointUpperLegR: limit lower=-0.698132 upper=+1.047 effort=90 velocity=10 -> lower=-1.047 upper=+0.698132 effort=90 velocity=10
