Commit message: 1

File: urdf/simbicon_urdf/flame4.urdf (robot description, URDF)
Before this commit: robot humanoid, 30 links, 29 joints
Links:
- added link world, mass 0
- added link y_prismatic, mass 0.01
- added link z_prismatic, mass 0.01
Joints:
- removed joint left_hip_motor
- removed joint left_knee_motor
- removed joint right_hip_motor
- removed joint right_knee_motor
- added joint fixed_RightupperLegToRight_Motor2_Gear: type fixed, parent upperLegCylinderR, child Right_Motor2_gear, origin xyz=0 -0.02 -0.1 rpy=0 0 0
- added joint fixed_upperLegToMotor1_Gear: type fixed, parent upperLegCylinderL, child Left_Motor1_gear, origin xyz=0 0.02 -0.1 rpy=0 0 0
- added joint fixed_upperLegToMotor2_Gear: type fixed, parent upperLegCylinderL, child Left_Motor2_gear, origin xyz=0 -0.02 -0.1 rpy=0 0 0
- added joint fixed_upperRightLegToRight_Motor1_Gear: type fixed, parent upperLegCylinderR, child Right_Motor1_gear, origin xyz=0 0.02 -0.1 rpy=0 0 0
- added joint torso_to_z: type continuous, parent z_prismatic, child body, origin xyz=0 0 1.4 rpy=0 0 0, axis 1 0 0
- added joint y_to_world: type prismatic, parent world, child y_prismatic, origin xyz=0 0 0 rpy=0 0 0, axis 0 1 0, limit lower=1 upper=-1 effort=0.0 velocity=1000.0
- added joint z_to_y: type prismatic, parent y_prismatic, child z_prismatic, origin xyz=0 0 0 rpy=0 0 0, axis 0 0 1, limit lower=1 upper=-1 effort=0.0 velocity=1000.0

Commit message: 111

File: urdf/simbicon_urdf/flame4.urdf (robot description, URDF)
Before this commit: robot humanoid, 33 links, 32 joints
Joints:
- joint torso_to_z: child body -> torso

Commit message: traj and ea

File: urdf/simbicon_urdf/flame4.urdf (robot description, URDF)
Before this commit: robot humanoid, 33 links, 32 joints
Links:
- removed link Left_AnkleMotor_Gear
- removed link Left_Ankle_motor
- removed link Left_Motor1_gear
- removed link Left_Motor1_motor
- removed link Left_Motor2_gear
- removed link Left_Motor2_motor
- removed link Right_AnkleMotor_Gear
- removed link Right_Ankle_motor
- removed link Right_Motor1_gear
- removed link Right_Motor1_motor
- removed link Right_Motor2_gear
- removed link Right_Motor2_motor
- removed link torso
- removed link y_prismatic
- added link x_prismatic, mass 0.01
Joints:
- removed joint fixed_Left_AnkleMotor_GearToLeft_Ankle_motor
- removed joint fixed_Motor1_GearToMotor1_Motor
- removed joint fixed_Motor2_GearToMotor2_Motor
- removed joint fixed_Right_AnkleMotor_GearToRight_Ankle_motor
- removed joint fixed_Right_Motor1_GearToRight_Motor1_Motor
- removed joint fixed_Right_Motor2_GearToRight_Motor2_Motor
- removed joint fixed_RightupperLegToRight_Motor2_Gear
- removed joint fixed_lowerLegBridgeLToLeft_AnkleMotor_Gear
- removed joint fixed_lowerLegBridgeRToRight_AnkleMotor_Gear
- removed joint fixed_upperLegToMotor1_Gear
- removed joint fixed_upperLegToMotor2_Gear
- removed joint fixed_upperRightLegToRight_Motor1_Gear
- removed joint torsoBody
- removed joint y_to_world
- added joint x_to_world: type prismatic, parent world, child x_prismatic, origin xyz=0 0 0 rpy=0 0 0, axis 1 0 0, limit lower=10 upper=-10 effort=0.0 velocity=1000.0
- joint jointHipL: parent torso -> body
- joint jointHipR: parent torso -> body
- joint torso_to_z: axis 1 0 0 -> 0 1 0; child torso -> body; limit (none) -> lower=10 upper=-10 effort=0.0 velocity=1000.0; origin xyz=0 0 1.4 rpy=0 0 0 -> xyz=0 0 0 rpy=0 0 0; type continuous -> revolute
- joint z_to_y: limit lower=1 upper=-1 effort=0.0 velocity=1000.0 -> lower=10 upper=-10 effort=0.0 velocity=1000.0; parent y_prismatic -> x_prismatic

File: urdf/simbicon_urdf/flame5.urdf (robot description, URDF)
Before this commit: robot humanoid, 30 links, 29 joints
Links:
- removed link Left_AnkleMotor_Gear
- removed link Left_Ankle_motor
- removed link Left_Motor1_gear
- removed link Left_Motor1_motor
- removed link Left_Motor2_gear
- removed link Left_Motor2_motor
- removed link Right_AnkleMotor_Gear
- removed link Right_Ankle_motor
- removed link Right_Motor1_gear
- removed link Right_Motor1_motor
- removed link Right_Motor2_gear
- removed link Right_Motor2_motor
- removed link torso
- added link world, mass 0
- added link x_prismatic, mass 0.01
- added link z_prismatic, mass 0.01
- link body: mass 5.6 -> 5.81
- link lowerlegCylinderL: geometry visual cylinder length=0.04 radius=0.01
- link upperLegBridgeL: geometry collision box size=0.1 0.05 0.32; visual box size=0.1 0.05 0.32
- link upperLegBridgeR: geometry collision box size=0.1 0.05 0.32; visual box size=0.1 0.05 0.32
Joints:
- removed joint fixed_Left_AnkleMotor_GearToLeft_Ankle_motor
- removed joint fixed_Motor1_GearToMotor1_Motor
- removed joint fixed_Motor2_GearToMotor2_Motor
- removed joint fixed_Right_AnkleMotor_GearToRight_Ankle_motor
- removed joint fixed_Right_Motor1_GearToRight_Motor1_Motor
- removed joint fixed_Right_Motor2_GearToRight_Motor2_Motor
- removed joint fixed_RightupperLegToRight_Motor2_Gear
- removed joint fixed_lowerLegBridgeLToLeft_AnkleMotor_Gear
- removed joint fixed_lowerLegBridgeRToRight_AnkleMotor_Gear
- removed joint fixed_upperLegToMotor1_Gear
- removed joint fixed_upperLegToMotor2_Gear
- removed joint fixed_upperRightLegToRight_Motor1_Gear
- removed joint torsoBody
- added joint torso_to_z: type revolute, parent z_prismatic, child body, origin xyz=0 0 0 rpy=0 0 0, axis 0 1 0, limit lower=10 upper=-10 effort=0.0 velocity=1000.0
- added joint x_to_world: type prismatic, parent world, child x_prismatic, origin xyz=0 0 0 rpy=0 0 0, axis 1 0 0, limit lower=10 upper=-10 effort=0.0 velocity=1000.0
- added joint z_to_y: type prismatic, parent x_prismatic, child z_prismatic, origin xyz=0 0 0 rpy=0 0 0, axis 0 0 1, limit lower=10 upper=-10 effort=0.0 velocity=1000.0
- joint jointHipL: origin xyz=0 0.0 0.0 rpy=0 0 0 -> xyz=0 0.0 -0.15 rpy=0 0 0; parent torso -> body
- joint jointHipR: origin xyz=0 0.0 0.0 rpy=0 0 0 -> xyz=0 0.0 -0.15 rpy=0 0 0; parent torso -> body

File: urdf/simbicon_urdf/test.urdf (robot description, URDF)
Before this commit: robot test, 5 links, 4 joints
Links:
- removed link base
- added link hinge, mass 0.00001; visual cylinder length=0.02 radius=0.005
- added link motor, mass 0.59; collision cylinder length=0.066714 radius=0.02; visual cylinder length=0.066714 radius=0.02
- link upperLegCylinderR: mass 0 -> 0.0000001
Joints:
- removed joint root
- added joint hingeToMotor: type revolute, parent hinge, child motor, origin xyz=0 0 -0.01 rpy=0 0 0, axis 0 0 1, limit lower=-1.57 upper=1.57 effort=90 velocity=672
- added joint legToHinge: type fixed, parent upperLegCylinderR, child hinge, origin xyz=0 0 -0.1 rpy=0 0 0, axis 0 0 1
- joint jointLowerLegR: limit lower=0 upper=1.570796 effort=90 velocity=10 -> lower=0 upper=1.570796 effort=90 velocity=672

File: urdf/simbicon_urdf/test5.urdf (robot description, URDF)
Before this commit: robot test, 2 links, 1 joints
Links:
- link lowerLegBridgeR: geometry collision box size=0.05 0.05 0.28; visual box size=0.05 0.05 0.28
- link upperLegBridgeR: mass 100.94 -> 1.94; geometry collision box size=0.1 0.05 0.3155; visual box size=0.1 0.05 0.3155

Commit message: supervised learning

File: urdf/simbicon_urdf/flame4.urdf (robot description, URDF)
Before this commit: robot humanoid, 20 links, 19 joints
Links:
- removed link world
- removed link x_prismatic
- removed link z_prismatic
- link body: mass 5.6 -> 5.81
- link lowerlegCylinderL: geometry visual cylinder length=0.04 radius=0.01
- link upperLegBridgeL: geometry collision box size=0.1 0.05 0.32; visual box size=0.1 0.05 0.32
- link upperLegBridgeR: geometry collision box size=0.1 0.05 0.32; visual box size=0.1 0.05 0.32
Joints:
- removed joint torso_to_z
- removed joint x_to_world
- removed joint z_to_y
- joint jointHipL: origin xyz=0 0.0 0.0 rpy=0 0 0 -> xyz=0 0.0 -0.15 rpy=0 0 0; type revolute -> fixed
- joint jointHipR: origin xyz=0 0.0 0.0 rpy=0 0 0 -> xyz=0 0.0 -0.15 rpy=0 0 0; type revolute -> fixed
- joint jointUpperLegL: limit lower=-0.174533 upper=+0.174533 effort=10 velocity=10 -> lower=-0.523599 upper=+1.22173 effort=10 velocity=10
- joint jointUpperLegR: limit lower=-0.698132 upper=+1.047 effort=90 velocity=10 -> lower=-1.047 upper=+0.698132 effort=90 velocity=10
